File: telemetry-node.kicad_pcb (KiCad board)
At the start: 4 copper layers, 44.5 x 57.7 mm, 84 parts, among them IC1 TLV62569DBVR, IC2 USBLC6-2P6, J1 53047-0710, J11 USB_B_Micro, J14 S1, J15 S2, J2 SWD, J3 53048-0210, J4 53048-0210, J5 53047-0410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

Commit message: Fixed things
Connections:
- J11 pad 6: unconnected-(J11-Shield-Pad6)_2 -> GND
Routing:
- net GND: track 84.9 -> 85.4 mm, vias 52 -> 63

Commit message: Added temp
Other:
- board text added: "v1.2.0"
Changed lines of the file:
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@@
 	)
 	(gr_text "STM32F103"
-		(at 227.25 68.5 90)
+		(at 227.25 70 90)
 		(layer "F.SilkS")
 		(effects
@@
 		)
 	)
+	(gr_text "v1.2.0"
+		(at 227.1 60.7 90)
+		(layer "F.SilkS")
+		(effects
+			(font
+				(size 1 1)
+				(thickness 0.15)
+			)
+			(justify left bottom)
+		)
+	)
 	(gr_text "GPIOs"
 		(at 213.95 55.75 90)
@@
 	)
 	(gr_text "Quang."
-		(at 227 74.6 90)
-		(layer "F.SilkS")
-		(effects
+		(at 227 75.7 90)
+		(layer "F.SilkS")
+		(effects
