File: telemetry-node.kicad_pcb (KiCad board)
At the start: 4 copper layers, 44.5 x 57.7 mm, 84 parts, among them IC1 TLV62569DBVR, IC2 USBLC6-2P6, J1 53047-0710, J11 USB_B_Micro, J14 S1, J15 S2, J2 SWD, J3 53048-0210, J4 53048-0210, J5 53047-0410, J6 Conn_01x06_Pin, U1 STM32F103C4Tx, U2 TJA1051TK-3, Y1 16MHz

Commit message: Commit
Connections:
- J6 pad 3: /PA1 -> /PA2
- J6 pad 4: /PA2 -> /PA1
Routing:
- net /PA1: track 17.2 -> 18.0 mm
- net /PA2: track 15.4 -> 14.6 mm, vias 0 -> 1
Other:
- board text added: "v1.2.1"
- board text removed: "v1.2.0"
Changed lines of the file:
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@@
 			(layers "*.Cu" "*.Mask")
 			(remove_unused_layers no)
-			(net 60 "/PA1")
+			(net 63 "/PA2")
 			(pinfunction "Pin_3")
 			(pintype "passive")
@@
 			(layers "*.Cu" "*.Mask")
 			(remove_unused_layers no)
-			(net 63 "/PA2")
+			(net 60 "/PA1")
 			(pinfunction "Pin_4")
 			(pintype "passive")
@@
 		)
 	)
-	(gr_text "v1.2.0"
+	(gr_text "v1.2.1"
 		(at 227.1 60.7 90)
 		(layer "F.SilkS")
@@
 	)
 	(segment
-		(start 215.849 64.551)
-		(end 215.849 63.8339)
-		(width 0.2)
-		(layer "F.Cu")
-		(net 60)
-	)
-	(segment
-		(start 213.75 66.65)
-		(end 215.849 64.551)
+		(start 217.599 62.0839)
+		(end 217.599 58.151)
 		(width 0.2)
 		(layer "F.Cu")
@@
 	)
 	(segment
-		(start 219.9 56.8829)
-		(end 219.9 53.85)
+		(start 217.599 58.151)
+		(end 221.9 53.85)
 		(width 0.2)
 		(layer "F.Cu")
@@
 	)
 	(segment
-		(start 217.599 59.1839)
-		(end 219.9 56.8829)
+		(start 213.75 66.65)
+		(end 215.849 64.551)
 		(width 0.2)
 		(layer "F.Cu")
@@
 	)
 	(segment
-		(start 214 67.05)
-		(end 213.75 66.8)
+		(start 215.849 63.8339)
+		(end 217.599 62.0839)
 		(width 0.2)
 		(layer "F.Cu")
@@
 	)
 	(segment
-		(start 215.3375 67.05)
-		(end 214 67.05)
+		(start 215.849 64.551)
+		(end 215.849 63.8339)
 		(width 0.2)
 		(layer "F.Cu")
@@
 	)
 	(segment
-		(start 217.599 62.0839)
-		(end 217.599 59.1839)
+		(start 215.3375 67.05)
+		(end 214 67.05)
 		(width 0.2)
 		(layer "F.Cu")
@@
 	)
 	(segment
-		(start 215.849 63.8339)
-		(end 217.599 62.0839)
+		(start 214 67.05)
+		(end 213.75 66.8)
 		(width 0.2)
 		(layer "F.Cu")
@@
 	)
 	(segment
-		(start 216.25 65.6375)
-		(end 216.25 64)
+		(start 215.3375 66.55)
+		(end 216.25 65.6375)
 		(width 0.2)
 		(layer "F.Cu")
@@
 	)
 	(segment
-		(start 218 59.35)
-		(end 221.9 55.45)
+		(start 216.25 64)
+		(end 218 62.25)
 		(width 0.2)
 		(layer "F.Cu")
@@
 	)
 	(segment
-		(start 218 62.25)
-		(end 218 59.35)
+		(start 216.25 65.6375)
+		(end 216.25 64)
 		(width 0.2)
 		(layer "F.Cu")
@@
 	)
 	(segment
-		(start 215.3375 66.55)
-		(end 216.25 65.6375)
+		(start 218 59.3)
+		(end 219.8 57.5)
 		(width 0.2)
 		(layer "F.Cu")
@@
 	)
 	(segment
-		(start 221.9 55.45)
-		(end 221.9 53.85)
+		(start 218 62.25)
+		(end 218 59.3)
 		(width 0.2)
 		(layer "F.Cu")
 		(net 63)
 	)
+	(via
+		(at 219.8 57.5)
+		(size 0.6)
+		(drill 0.3)
+		(layers "F.Cu" "B.Cu")
+		(net 63)
+	)
 	(segment
-		(start 216.25 64)
-		(end 218 62.25)
+		(start 219.9 57.4)
+		(end 219.9 53.85)
 		(width 0.2)
-		(layer "F.Cu")
+		(layer "B.Cu")
+		(net 63)
+	)
+	(segment
+		(start 219.8 57.5)
+		(end 219.9 57.4)
+		(width 0.2)
+		(layer "B.Cu")
 		(net 63)
 	)
