File: telemetry-node.kicad_sch (KiCad schematic)
At the start: 67 parts, among them IC2 USBLC6-2P6, J1 53047-0710, J11 USB_B_Micro, J14 S1, J15 S2, J2 SWD, J4 53048-0210, J5 53047-0410, J6 Conn_01x06_Pin, U1 STM32F103C4Tx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

Commit message: Fixed things
Connections:
- net GND: now also J11.6 (Shield)
- no-connect marks 8 -> 7
Changed lines of the file:
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@@
+	)
+	(junction
+		(at 304.8 59.69)
+		(diameter 0)
+		(color 0 0 0 0)
 	)
 	(junction
@@
 	)
 	(no_connect
-		(at 302.26 57.15)
-	)
-	(no_connect
 		(at 128.27 104.14)
 	)
@@
 	(wire
 		(pts
+			(xy 302.26 59.69) (xy 304.8 59.69)
+		)
+		(stroke
+			(width 0)
+			(type default)
+		)
+	)
+	(wire
+		(pts
 			(xy 311.15 105.41) (xy 311.15 116.84)
 		)
@@
 	(wire
 		(pts
-			(xy 304.8 57.15) (xy 304.8 62.23)
+			(xy 304.8 57.15) (xy 304.8 59.69)
 		)
 		(stroke
@@
 	(wire
 		(pts
+			(xy 304.8 59.69) (xy 304.8 62.23)
+		)
+		(stroke
+			(width 0)
+			(type default)
+		)
+	)
+	(wire
+		(pts
 			(xy 74.93 238.76) (xy 80.01 238.76)
 		)
@@
 		)
 		(stroke
+			(width 0)
+			(type default)
+		)
+	)
+	(wire
+		(pts
+			(xy 302.26 57.15) (xy 302.26 59.69)
+		)
+		(stroke
