File: telemetry-node.kicad_sch (KiCad schematic)
At the start: 67 parts, among them IC2 USBLC6-2P6, J1 53047-0710, J11 USB_B_Micro, J14 S1, J15 S2, J2 SWD, J4 53048-0210, J5 53047-0410, J6 Conn_01x06_Pin, U1 STM32F103C4Tx, U2 TJA1051TK-3, Y1 16MHz

Commit message: Commit
Connections:
- net PA1: now also J6.4 (Pin_4); no longer J6.3 (Pin_3)
- net PA2: now also J6.3 (Pin_3); no longer J6.4 (Pin_4)
Changed lines of the file:
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@@
 	)
 	(label "PA2"
-		(at 306.07 227.33 0)
+		(at 306.07 224.79 0)
 		(effects
 			(font
@@
 	)
 	(label "PA1"
-		(at 306.07 224.79 0)
-		(effects
-			(font
+		(at 306.07 227.33 0)
+		(effects
+			(font
